File: p0001-001_test-board.kicad_pcb (KiCad board)
At the start: 2 copper layers, 100 x 100 mm, 5 parts

Commit message: Testing wut libraries
Parts:
- added CN1: U77-A1114-30L1, Connector_WUT:Amphenol_U77-A1114-30L1, F.Cu at (165.0, 98.7)
